File: hackpadpcb/_autosave-hackpadd.kicad_pcb (KiCad board)
At the start: 2 copper layers, 81 x 67.3 mm, 9 parts, among them SW1 SW_Push, SW2 SW_Push, SW3 SW_Push, SW4 SW_Push, SW5 RotaryEncoder, SW6 SW_Push, U1 XIAO-RP2040-DIP, U2 OLED

Commit message: finish schem and pcb
Routing:
- net GND: track 153.9 -> 158.7 mm
Changed lines of the file:
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@@
 	(segment
 		(start 181.13375 104.4575)
-		(end 183.8325 107.15625)
+		(end 185.89625 104.4575)
 		(width 0.2)
 		(layer "F.Cu")
@@
 	)
 	(segment
-		(start 183.8325 107.15625)
-		(end 200.18375 107.15625)
-		(width 0.2)
-		(layer "F.Cu")
-		(net 1)
-	)
-	(segment
 		(start 155.31862 108.563684)
 		(end 157.19275 108.563684)
@@
 		(width 0.2)
 		(layer "F.Cu")
+		(net 1)
+	)
+	(segment
+		(start 185.89625 104.4575)
+		(end 200.18375 118.745)
+		(width 0.2)
+		(layer "F.Cu")
